File: hardware/phased-array-controller-v1/phased-array-controller-v1.kicad_sch (KiCad schematic)
At the start: 0 parts

Commit message: updates
Parts:
- added IC1, IC2, IC3, IC4, IC5: WP4U+, QFN51P300X300X89-13N, symbol phased-array:WP4U+
- added J1: Conn_Coaxial, Connector_Coaxial:SMA_Amphenol_901-144_Vertical, symbol Connector:Conn_Coaxial
- added R1: 10k, Resistor_SMD:R_0603_1608Metric, symbol Device:R_Small
- added R2: 12k, Resistor_SMD:R_0603_1608Metric, symbol Device:R_Small
- added U1: SKY13330-397LF, SKY13330397LF, symbol phased-array:SKY13330-397LF
Connections:
- new net: IC1.6 (PORT_3), IC2.2 (SUM_PORT)
- new net: IC4.12 (PORT_1), U1.2 (RF1)
- new net: R1.1, U1.8 (ENABLE)
- new net: R1.2, R2.1, U1.9 (VBATT)
- new net: IC1.12 (PORT_1), IC4.2 (SUM_PORT)
- new net: IC1.10 (PORT_2), IC3.2 (SUM_PORT)
- new net: IC1.4 (PORT_4), IC5.2 (SUM_PORT)
- new net: IC1.2 (SUM_PORT), J1.1 (In)
- new net GND: IC1.1 (GROUND_1), IC1.11 (GROUND_7), IC1.13 (GROUND_8), IC1.3 (GROUND_2), IC1.5 (GROUND_3), IC1.7 (GROUND_4), IC1.8 (GROUND_5), IC1.9 (GROUND_6), IC2.1 (GROUND_1), IC2.11 (GROUND_7), IC2.13 (GROUND_8), IC2.3 (GROUND_2), IC2.5 (GROUND_3), IC2.7 (GROUND_4), IC2.8 (GROUND_5), IC2.9 (GROUND_6), IC3.1 (GROUND_1), IC3.11 (GROUND_7), IC3.13 (GROUND_8), IC3.3 (GROUND_2), IC3.5 (GROUND_3), IC3.7 (GROUND_4), IC3.8 (GROUND_5), IC3.9 (GROUND_6), IC4.1 (GROUND_1), IC4.11 (GROUND_7), IC4.13 (GROUND_8), IC4.3 (GROUND_2), IC4.5 (GROUND_3), IC4.7 (GROUND_4), IC4.8 (GROUND_5), IC4.9 (GROUND_6), IC5.1 (GROUND_1), IC5.11 (GROUND_7), IC5.13 (GROUND_8), IC5.3 (GROUND_2), IC5.5 (GROUND_3), IC5.7 (GROUND_4), IC5.8 (GROUND_5), IC5.9 (GROUND_6), J1.2 (Ext), R2.2, U1.1 (GND), U1.10 (GND_5), U1.12 (GND_6), U1.13 (EP), U1.3 (GND_2), U1.4 (GND_3), U1.6 (GND_4)

Commit message: updates
Parts:
- removed IC1: WP4U+, QFN51P300X300X89-13N, symbol phased-array:WP4U+
- removed R1: 10k, Resistor_SMD:R_0603_1608Metric, symbol Device:R_Small
- removed R2: 12k, Resistor_SMD:R_0603_1608Metric, symbol Device:R_Small
- removed U1: SKY13330-397LF, SKY13330397LF, symbol phased-array:SKY13330-397LF
- added U1: WP4U+, QFN51P300X300X89-13N, symbol phased-array:WP4U+
- renumbered IC4 to U2, IC3 to U3, IC2 to U4, IC5 to U5
Connections:
- net GND: now also U1.1 (GROUND_1), U1.11 (GROUND_7), U1.13 (GROUND_8), U1.3 (GROUND_2), U1.5 (GROUND_3), U1.7 (GROUND_4), U1.8 (GROUND_5), U1.9 (GROUND_6)
- net Element9-12/E10: now reaches U4.10 (PORT_2)
- net Element9-12/E9: now reaches U4.12 (PORT_1)
- net at U4.2 (SUM_PORT): now also U1.6 (PORT_3)
- net Element9-12/E12: now reaches U4.4 (PORT_4)
- net Element9-12/E11: now reaches U4.6 (PORT_3)
- net Element1-4/E1: now reaches U2.12 (PORT_1)
- net Element1-4/E2: now reaches U2.10 (PORT_2)
- net at U2.2 (SUM_PORT): now also U1.12 (PORT_1)
- net Element1-4/E4: now reaches U2.4 (PORT_4)
- net Element1-4/E3: now reaches U2.6 (PORT_3)
- net Element5-8/E6: now reaches U3.10 (PORT_2)
- net Element5-8/E5: now reaches U3.12 (PORT_1)
- net at U3.2 (SUM_PORT): now also U1.10 (PORT_2)
- net Element5-8/E8: now reaches U3.4 (PORT_4)
- net Element5-8/E7: now reaches U3.6 (PORT_3)
- net Element13-16/E14: now reaches U5.10 (PORT_2)
- net Element13-16/E13: now reaches U5.12 (PORT_1)
- net at U5.2 (SUM_PORT): now also U1.4 (PORT_4)
- net Element13-16/E16: now reaches U5.4 (PORT_4)
- net Element13-16/E15: now reaches U5.6 (PORT_3)
- net at J1.1 (In): now also U1.2 (SUM_PORT)
Other:
- added sheet Element1-4 (E1-4.kicad_sch)
- added sheet Element13-16 (E13-16.kicad_sch)
- added sheet Element5-8 (E5-8.kicad_sch)
- added sheet Element9-12 (E9-12.kicad_sch)
- moved on the sheet: J1, U2, U3, U4, U5
